File: lab4/Excercise1/Excercise1.kicad_sch (KiCad schematic)
At the start: 6 parts, among them SW1 SW_SPDT

Commit message: Excercisee 1 and 2 for lab 6
Parts:
- C1: footprint (none) -> Capacitor_THT:C_Radial_D5.0mm_H11.0mm_P2.00mm
- D1: footprint (none) -> LED_THT:LED_D5.0mm
- R1: renamed from R2; footprint (none) -> Resistor_THT:R_Axial_DIN0516_L15.5mm_D5.0mm_P20.32mm_Horizontal
- R2: renamed from R1; footprint (none) -> Resistor_THT:R_Axial_DIN0516_L15.5mm_D5.0mm_P20.32mm_Horizontal
- SW1: footprint (none) -> Button_Switch_THT:SW_E-Switch_EG1224_SPDT_Angled
- V1: footprint (none) -> Connector_JST:JST_PH_B2B-PH-K_1x02_P2.00mm_Vertical
Connections:
- no-connect marks 0 -> 2
Other:
- added sheet Lab 4 Sheet (lab4.kicad_sch)
Changed lines of the file:
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@@
   (junction (at 153.67 77.47) (diameter 0) (color 0 0 0 0)
   )
+  (no_connect (at 165.1 118.11))
+  (no_connect (at 152.4 72.39))
   (wire (pts (xy 177.8 101.6) (xy 177.8 104.14))
     (stroke (width 0) (type default) (color 0 0 0 0))
@@
     (stroke (width 0) (type default) (color 0 0 0 0))
   )
+  (wire (pts (xy 148.59 72.39) (xy 152.4 72.39))
+    (stroke (width 0) (type default) (color 0 0 0 0))
+  )
   (symbol (lib_id "pspice:R") (at 124.46 74.93 90) (unit 1)
     (in_bom yes) (on_board yes) (fields_autoplaced)
-    (property "Reference" "R1" (id 0) (at 124.46 68.58 90))
+    (property "Reference" "R2" (id 0) (at 124.46 68.58 90))
     (property "Value" "2.2 kOhm" (id 1) (at 124.46 71.12 90))
-    (property "Footprint" "" (id 2) (at 124.46 74.93 0)
+    (property "Footprint" "Resistor_THT:R_Axial_DIN0516_L15.5mm_D5.0mm_P20.32mm_Horizontal" (id 2) (at 124.46 74.93 0)
       (effects (font (size 1.27 1.27)) hide)
     )
@@
       (effects (font (size 1.27 1.27)) (justify right))
     )
-    (property "Footprint" "" (id 2) (at 177.8 97.79 0)
+    (property "Footprint" "LED_THT:LED_D5.0mm" (id 2) (at 177.8 97.79 0)
       (effects (font (size 1.27 1.27)) hide)
     )
@@
   (symbol (lib_id "pspice:R") (at 177.8 83.82 0) (unit 1)
     (in_bom yes) (on_board yes) (fields_autoplaced)
-    (property "Reference" "R2" (id 0) (at 180.34 82.5499 0)
+    (property "Reference" "R1" (id 0) (at 180.34 82.5499 0)
       (effects (font (size 1.27 1.27)) (justify left))
     )
@@
       (effects (font (size 1.27 1.27)) (justify left))
     )
-    (property "Footprint" "" (id 2) (at 177.8 83.82 0)
+    (property "Footprint" "Resistor_THT:R_Axial_DIN0516_L15.5mm_D5.0mm_P20.32mm_Horizontal" (id 2) (at 177.8 83.82 0)
       (effects (font (size 1.27 1.27)) hide)
     )
@@
     (property "Reference" "V1" (id 0) (at 107.315 69.85 0))
     (property "Value" "9 V" (id 1) (at 107.315 72.39 0))
-    (property "Footprint" "" (id 2) (at 106.68 74.93 0)
+    (property "Footprint" "Connector_JST:JST_PH_B2B-PH-K_1x02_P2.00mm_Vertical" (id 2) (at 106.68 74.93 0)
       (effects (font (size 1.27 1.27)) hide)
     )
@@
     (property "Reference" "SW1" (id 0) (at 143.51 67.31 0))
     (property "Value" "SW_SPDT" (id 1) (at 143.51 69.85 0))
-    (property "Footprint" "" (id 2) (at 143.51 74.93 0)
+    (property "Footprint" "Button_Switch_THT:SW_E-Switch_EG1224_SPDT_Angled" (id 2) (at 143.51 74.93 0)
       (effects (font (size 1.27 1.27)) hide)
     )
@@
       (effects (font (size 1.27 1.27)) (justify left))
     )
-    (property "Footprint" "" (id 2) (at 154.6352 93.98 0)
+    (property "Footprint" "Capacitor_THT:C_Radial_D5.0mm_H11.0mm_P2.00mm" (id 2) (at 154.6352 93.98 0)
       (effects (font (size 1.27 1.27)) hide)
     )
@@
     (pin "2")
   )
+  (sheet (at 99.06 63.5) (size 93.98 45.72) (fields_autoplaced)
+    (stroke (width 0.1524) (type solid) (color 0 0 0 0))
+    (fill (color 0 0 0 0.0000))
+    (property "Sheet name" "Lab 4 Sheet" (id 0) (at 99.06 62.7884 0)
+      (effects (font (size 1.27 1.27)) (justify left bottom))
+    )
+    (property "Sheet file" "lab4.kicad_sch" (id 1) (at 99.06 109.8046 0)
+      (effects (font (size 1.27 1.27)) (justify left top))
+    )
+  )
   (sheet_instances
     (path "/" (page "1"))
+    (path "/62448543-fbb0-4641-9f76-b1edb35a0427" (page "2"))
   )
   (symbol_instances
     (path "/f962a014-e4f8-4779-8028-ccd04dcbb9d8"
-      (reference "C1") (unit 1) (value "4.7 uF") (footprint "")
+      (reference "C1") (unit 1) (value "4.7 uF") (footprint "Capacitor_THT:C_Radial_D5.0mm_H11.0mm_P2.00mm")
     )
     (path "/45d42230-1d16-47dc-a8bb-5ad973e5fe35"
-      (reference "D1") (unit 1) (value "LED") (footprint "")
+      (reference "D1") (unit 1) (value "LED") (footprint "LED_THT:LED_D5.0mm")
+    )
+    (path "/7e475528-7f47-41c6-87ce-6615f495761d"
+      (reference "R1") (unit 1) (value "20 kOhm") (footprint "Resistor_THT:R_Axial_DIN0516_L15.5mm_D5.0mm_P20.32mm_Horizontal")
     )
     (path "/0e62f881-95fa-4aab-80c9-4fba57a70255"
-      (reference "R1") (unit 1) (value "2.2 kOhm") (footprint "")
-    )
-    (path "/7e475528-7f47-41c6-87ce-6615f495761d"
-      (reference "R2") (unit 1) (value "20 kOhm") (footprint "")
+      (reference "R2") (unit 1) (value "2.2 kOhm") (footprint "Resistor_THT:R_Axial_DIN0516_L15.5mm_D5.0mm_P20.32mm_Horizontal")
     )
     (path "/f2046d4f-d1af-4793-a754-9631a86962a6"
-      (reference "SW1") (unit 1) (value "SW_SPDT") (footprint "")
+      (reference "SW1") (unit 1) (value "SW_SPDT") (footprint "Button_Switch_THT:SW_E-Switch_EG1224_SPDT_Angled")
     )
     (path "/f124860c-9100-4789-8e88-25142d05c77e"
-      (reference "V1") (unit 1) (value "9 V") (footprint "")
+      (reference "V1") (unit 1) (value "9 V") (footprint "Connector_JST:JST_PH_B2B-PH-K_1x02_P2.00mm_Vertical")
     )
   )
