File: lab4/Excercise2/Excercise2.kicad_sch (KiCad schematic)
At the start: 10 parts, among them J1 J1, U1 NE555D

Commit message: Excercisee 1 and 2 for lab 6
Parts:
- C1: footprint (none) -> Capacitor_Tantalum_SMD:CP_EIA-3216-18_Kemet-A_Pad1.58x1.35mm_HandSolder
- C2: footprint (none) -> Capacitor_SMD:C_0805_2012Metric_Pad1.18x1.45mm_HandSolder
- D1, D2: footprint (none) -> LED_SMD:LED_1206_3216Metric_Pad1.42x1.75mm_HandSolder
- J1: footprint (none) -> TerminalBlock:TerminalBlock_bornier-2_P5.08mm
- R1, R2, R3, R4: footprint (none) -> Resistor_SMD:R_0805_2012Metric_Pad1.20x1.40mm_HandSolder
Changed lines of the file:
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@@
   (junction (at 102.87 87.63) (diameter 0) (color 0 0 0 0)
   )
+  (junction (at 140.97 123.19) (diameter 0) (color 0 0 0 0)
+  )
   (junction (at 121.92 123.19) (diameter 0) (color 0 0 0 0)
   )
@@
   (junction (at 102.87 107.95) (diameter 0) (color 0 0 0 0)
   )
-  (junction (at 140.97 123.19) (diameter 0) (color 0 0 0 0)
-  )
   (junction (at 175.26 77.47) (diameter 0) (color 0 0 0 0)
   )
@@
     (stroke (width 0) (type default) (color 0 0 0 0))
   )
+  (wire (pts (xy 140.97 123.19) (xy 148.59 123.19))
+    (stroke (width 0) (type default) (color 0 0 0 0))
+  )
   (wire (pts (xy 140.97 123.19) (xy 140.97 128.27))
     (stroke (width 0) (type default) (color 0 0 0 0))
@@
     (stroke (width 0) (type default) (color 0 0 0 0))
   )
-  (wire (pts (xy 140.97 123.19) (xy 148.59 123.19))
+  (wire (pts (xy 121.92 123.19) (xy 140.97 123.19))
     (stroke (width 0) (type default) (color 0 0 0 0))
   )
@@
   )
   (wire (pts (xy 175.26 105.41) (xy 175.26 115.57))
-    (stroke (width 0) (type default) (color 0 0 0 0))
-  )
-  (wire (pts (xy 121.92 123.19) (xy 140.97 123.19))
     (stroke (width 0) (type default) (color 0 0 0 0))
   )
@@
       (effects (font (size 1.27 1.27)) (justify right) hide)
     )
-    (property "Footprint" "" (id 2) (at 146.05 69.85 0)
+    (property "Footprint" "TerminalBlock:TerminalBlock_bornier-2_P5.08mm" (id 2) (at 146.05 69.85 0)
       (effects (font (size 1.27 1.27)) hide)
     )
@@
       (effects (font (size 1.27 1.27)) (justify left))
     )
-    (property "Footprint" "" (id 2) (at 103.8352 123.19 0)
+    (property "Footprint" "Capacitor_Tantalum_SMD:CP_EIA-3216-18_Kemet-A_Pad1.58x1.35mm_HandSolder" (id 2) (at 103.8352 123.19 0)
       (effects (font (size 1.27 1.27)) hide)
     )
@@
   (symbol (lib_id "power:+9V") (at 148.59 82.55 0) (unit 1)
     (in_bom yes) (on_board yes) (fields_autoplaced)
-    (property "Reference" "#PWR?" (id 0) (at 148.59 86.36 0)
+    (property "Reference" "#PWR0103" (id 0) (at 148.59 86.36 0)
       (effects (font (size 1.27 1.27)) hide)
     )
@@
       (effects (font (size 1.27 1.27)) (justify left))
     )
-    (property "Footprint" "" (id 2) (at 101.092 96.52 90)
+    (property "Footprint" "Resistor_SMD:R_0805_2012Metric_Pad1.20x1.40mm_HandSolder" (id 2) (at 101.092 96.52 90)
       (effects (font (size 1.27 1.27)) hide)
     )
@@
   (symbol (lib_id "power:+9V") (at 146.05 59.69 0) (unit 1)
     (in_bom yes) (on_board yes) (fields_autoplaced)
-    (property "Reference" "#PWR?" (id 0) (at 146.05 63.5 0)
+    (property "Reference" "#PWR0104" (id 0) (at 146.05 63.5 0)
       (effects (font (size 1.27 1.27)) hide)
     )
@@
       (effects (font (size 1.27 1.27)) (justify left))
     )
-    (property "Footprint" "" (id 2) (at 173.482 81.28 90)
+    (property "Footprint" "Resistor_SMD:R_0805_2012Metric_Pad1.20x1.40mm_HandSolder" (id 2) (at 173.482 81.28 90)
       (effects (font (size 1.27 1.27)) hide)
     )
@@
   (symbol (lib_id "power:+9V") (at 175.26 57.15 0) (unit 1)
     (in_bom yes) (on_board yes) (fields_autoplaced)
-    (property "Reference" "#PWR?" (id 0) (at 175.26 60.96 0)
+    (property "Reference" "#PWR0106" (id 0) (at 175.26 60.96 0)
       (effects (font (size 1.27 1.27)) hide)
     )
@@
       (effects (font (size 1.27 1.27)) (justify left))
     )
-    (property "Footprint" "" (id 2) (at 122.8852 110.49 0)
+    (property "Footprint" "Capacitor_SMD:C_0805_2012Metric_Pad1.18x1.45mm_HandSolder" (id 2) (at 122.8852 110.49 0)
       (effects (font (size 1.27 1.27)) hide)
     )
@@
   (symbol (lib_id "power:GND") (at 148.59 59.69 180) (unit 1)
     (in_bom yes) (on_board yes)
-    (property "Reference" "#PWR?" (id 0) (at 148.59 53.34 0)
+    (property "Reference" "#PWR0105" (id 0) (at 148.59 53.34 0)
       (effects (font (size 1.27 1.27)) hide)
     )
@@
       (effects (font (size 1.27 1.27)) (justify right))
     )
-    (property "Footprint" "" (id 2) (at 175.26 119.38 0)
+    (property "Footprint" "LED_SMD:LED_1206_3216Metric_Pad1.42x1.75mm_HandSolder" (id 2) (at 175.26 119.38 0)
       (effects (font (size 1.27 1.27)) hide)
     )
@@
   (symbol (lib_id "power:+9V") (at 102.87 74.93 0) (unit 1)
     (in_bom yes) (on_board yes) (fields_autoplaced)
-    (property "Reference" "#PWR?" (id 0) (at 102.87 78.74 0)
+    (property "Reference" "#PWR0101" (id 0) (at 102.87 78.74 0)
       (effects (font (size 1.27 1.27)) hide)
     )
@@
       (effects (font (size 1.27 1.27)) (justify left))
     )
-    (property "Footprint" "" (id 2) (at 101.092 78.74 90)
+    (property "Footprint" "Resistor_SMD:R_0805_2012Metric_Pad1.20x1.40mm_HandSolder" (id 2) (at 101.092 78.74 90)
       (effects (font (size 1.27 1.27)) hide)
     )
@@
       (effects (font (size 1.27 1.27)) (justify right))
     )
-    (property "Footprint" "" (id 2) (at 175.26 60.96 0)
+    (property "Footprint" "LED_SMD:LED_1206_3216Metric_Pad1.42x1.75mm_HandSolder" (id 2) (at 175.26 60.96 0)
       (effects (font (size 1.27 1.27)) hide)
     )
@@
   (symbol (lib_id "power:GND") (at 140.97 128.27 0) (unit 1)
     (in_bom yes) (on_board yes) (fields_autoplaced)
-    (property "Reference" "#PWR?" (id 0) (at 140.97 134.62 0)
+    (property "Reference" "#PWR0102" (id 0) (at 140.97 134.62 0)
       (effects (font (size 1.27 1.27)) hide)
     )
@@
       (effects (font (size 1.27 1.27)) (justify left))
     )
-    (property "Footprint" "" (id 2) (at 173.482 101.6 90)
+    (property "Footprint" "Resistor_SMD:R_0805_2012Metric_Pad1.20x1.40mm_HandSolder" (id 2) (at 173.482 101.6 90)
       (effects (font (size 1.27 1.27)) hide)
     )
@@
   )
   (symbol_instances
+    (path "/bf7b73cf-0bc5-4c63-82e8-09a4b68565c7"
+      (reference "#PWR0101") (unit 1) (value "+9V") (footprint "")
+    )
+    (path "/dfad7b4b-c68e-4ba8-9137-1d755c33fd9b"
+      (reference "#PWR0102") (unit 1) (value "GND") (footprint "")
+    )
     (path "/5a1e8bbc-43bb-4f7d-9724-e4ef77d9f47f"
-      (reference "#PWR?") (unit 1) (value "+9V") (footprint "")
+      (reference "#PWR0103") (unit 1) (value "+9V") (footprint "")
     )
     (path "/6a97a7b6-f2cd-4a41-9dbb-a0d76ca03ce9"
-      (reference "#PWR?") (unit 1) (value "+9V") (footprint "")
+      (reference "#PWR0104") (unit 1) (value "+9V") (footprint "")
+    )
+    (path "/ae1fc28d-16bc-47ba-aafc-8fd9f4b4bfe4"
+      (reference "#PWR0105") (unit 1) (value "GND") (footprint "")
     )
     (path "/8e8aef23-20b0-4828-a1e3-a44e9869e7c0"
-      (reference "#PWR?") (unit 1) (value "+9V") (footprint "")
-    )
-    (path "/ae1fc28d-16bc-47ba-aafc-8fd9f4b4bfe4"
-      (reference "#PWR?") (unit 1) (value "GND") (footprint "")
-    )
-    (path "/bf7b73cf-0bc5-4c63-82e8-09a4b68565c7"
-      (reference "#PWR?") (unit 1) (value "+9V") (footprint "")
-    )
-    (path "/dfad7b4b-c68e-4ba8-9137-1d755c33fd9b"
-      (reference "#PWR?") (unit 1) (value "GND") (footprint "")
+      (reference "#PWR0106") (unit 1) (value "+9V") (footprint "")
     )
     (path "/53c4fb15-e6df-458d-819d-d76aef780685"
-      (reference "C1") (unit 1) (value "10uF") (footprint "")
+      (reference "C1") (unit 1) (value "10uF") (footprint "Capacitor_Tantalum_SMD:CP_EIA-3216-18_Kemet-A_Pad1.58x1.35mm_HandSolder")
     )
     (path "/8fc2dab2-684f-4f8b-8446-3b22efb6eb24"
-      (reference "C2") (unit 1) (value "0.01uF") (footprint "")
+      (reference "C2") (unit 1) (value "0.01uF") (footprint "Capacitor_SMD:C_0805_2012Metric_Pad1.18x1.45mm_HandSolder")
     )
     (path "/da14b71b-ee80-4534-bc8f-08c4f3c94064"
-      (reference "D1") (unit 1) (value "LED") (footprint "")
+      (reference "D1") (unit 1) (value "LED") (footprint "LED_SMD:LED_1206_3216Metric_Pad1.42x1.75mm_HandSolder")
     )
     (path "/bcd8bd2a-e9ac-4b74-81de-12a86d57f0e5"
-      (reference "D2") (unit 1) (value "LED") (footprint "")
+      (reference "D2") (unit 1) (value "LED") (footprint "LED_SMD:LED_1206_3216Metric_Pad1.42x1.75mm_HandSolder")
     )
     (path "/4f28160c-8830-429b-8985-e9b7a7049468"
-      (reference "J1") (unit 1) (value "J1") (footprint "")
+      (reference "J1") (unit 1) (value "J1") (footprint "TerminalBlock:TerminalBlock_bornier-2_P5.08mm")
     )
     (path "/c1d3a8ad-ea70-4fa3-b697-9d9ec5f8769b"
-      (reference "R1") (unit 1) (value "1k") (footprint "")
+      (reference "R1") (unit 1) (value "1k") (footprint "Resistor_SMD:R_0805_2012Metric_Pad1.20x1.40mm_HandSolder")
     )
     (path "/5a6d8565-779b-44fd-b511-57b8f3afbc35"
-      (reference "R2") (unit 1) (value "10k") (footprint "")
+      (reference "R2") (unit 1) (value "10k") (footprint "Resistor_SMD:R_0805_2012Metric_Pad1.20x1.40mm_HandSolder")
     )
     (path "/73f1bf52-c45e-4a3c-b637-362f21f0479d"
-      (reference "R3") (unit 1) (value "1k") (footprint "")
+      (reference "R3") (unit 1) (value "1k") (footprint "Resistor_SMD:R_0805_2012Metric_Pad1.20x1.40mm_HandSolder")
     )
     (path "/e6b7295f-3600-4335-9774-b4f7006efaf1"
-      (reference "R4") (unit 1) (value "1K") (footprint "")
+      (reference "R4") (unit 1) (value "1K") (footprint "Resistor_SMD:R_0805_2012Metric_Pad1.20x1.40mm_HandSolder")
     )
     (path "/cc50ccef-557e-4f8b-a57f-0f5fb5268f9c"
